File: Hardware/HadesNT/HadesNT.kicad_pcb (KiCad board)
At the start: 4 copper layers, 80 x 50 mm, 99 parts, among them J1 USB_B_Micro, J10 Conn_02x08_Odd_Even, J11 Conn_01x08, J2 Conn_01x02, J3 Conn_02x05_Odd_Even, J4 Conn_01x04, J5 Conn_01x04, J6 Conn_01x04, J7 Conn_01x04, J8 Conn_01x06, J9 Conn_01x02, Q1 AO4407A, Q2 MMBT3904, Q3 MMBT3904, Q4 MMBT3904, Q5 MMBT3904, Q6 MMBT3904, Q7 MMBT3904, U1 INA219AIDCNR, U2 MP2451DT-LF-Z, U3 SRV05-4, U4 W25Q128JVS, U5 BMP280, U6 BMX055, U7 STM32H750VBT6, Y1 16 MHz

Commit message: EKF STM32F4 testbed.
Parts:
- moved J9 0.30 mm to (94.7, 35.5)
Connections:
- net TIM3_CH1 renamed TIM8_CH1
- net TIM3_CH2 renamed TIM8_CH2
- net TIM3_CH3 renamed TIM8_CH3
- net TIM3_CH4 renamed TIM8_CH4
- U6 pad 10: Net-(U6-Pad10) -> MAG_INT
- U6 pad 2: MAG_INT -> MAGD_DRDY
- U7 pad 34: Net-(U7-Pad34) -> MAGD_DRDY
- U7 pad 35: Net-(U7-Pad35) -> MAG_INT
- U7 pad 7: GYR_INT -> Net-(U7-Pad7)
- U7 pad 8: ACC_INT -> Net-(U7-Pad8)
- U7 pad 81: Net-(U7-Pad81) -> LED_A
- U7 pad 82: Net-(U7-Pad82) -> LED_B
- U7 pad 9: MAG_INT -> Net-(U7-Pad9)
- U7 pad 90: LED_A -> ACC_INT
- U7 pad 91: LED_B -> GYR_INT
Routing:
- net GYR_!CS: track 1.52 -> 40.2 mm, vias 1 -> 2
- net I2C2_SDA: track 3.51 -> 40.8 mm, vias 0 -> 2
- net I2C2_SCL: track 2.21 -> 36.3 mm, vias 0 -> 2
- net QSPI_!CS: track 0.00 -> 33.4 mm
- net ACC_INT: track 2.52 -> 32.7 mm, vias 0 -> 2
- net MAG_INT: track 2.50 -> 29.6 mm, vias 0 -> 2
- net MAG_!CS: track 1.66 -> 26.5 mm, vias 1 -> 2
- net MAGD_DRDY: track 0.00 -> 24.7 mm, vias 0 -> 2
- net GYR_INT: track 4.50 -> 27.1 mm, vias 0 -> 2
- net GND: track 138.0 -> 156.5 mm, vias 89 -> 192
- net ACC_!CS: track 4.01 -> 18.8 mm, vias 1 -> 2
- net LED_A: track 29.8 -> 37.2 mm, vias 0 -> 2
- net LED_B: track 34.0 -> 40.3 mm, vias 0 -> 2
- net SPI4_MISO: track 23.8 -> 28.3 mm
- net USB_D+: track 21.8 -> 22.9 mm
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Other:
- board text added: "ERR"
- board text added: "JLCJLCJLCJLC"
- board text added: "REV A"
- board text added: "VI-MMXX"
- board text added: "philsal.co.uk"
- board text removed: "FLT"

Commit message: Finished HadesNT.
Parts:
- added D8: RE, LED_SMD:LED_0603_1608Metric, F.Cu at (56.1, 29.5)
- added R25: 2k2, Resistor_SMD:R_0603_1608Metric, F.Cu at (59.1, 29.5)
- added SP1: SolderPad, TestPoint:TestPoint_Pad_2.0x2.0mm, B.Cu at (95.4, 33.8)
- added SP2: SolderPad, TestPoint:TestPoint_Pad_2.0x2.0mm, F.Cu at (95.4, 33.8)
- J6: value Conn_01x04 -> Conn_01x06; footprint Connector_JST:JST_GH_SM04B-GHS-TB_1x04-1MP_P1.25mm_Horizontal -> Connector_JST:JST_GH_SM06B-GHS-TB_1x06-1MP_P1.25mm_Horizontal
- J9: value Conn_01x02 -> Conn_01x08; footprint TerminalBlock_Phoenix:TerminalBlock_Phoenix_PT-1,5-2-3.5-H_1x02_P3.50mm_Horizontal -> Connector_JST:JST_GH_SM08B-GHS-TB_1x08-1MP_P1.25mm_Horizontal
- Q1: value AO4407A -> AO3401A; footprint AO4407A:SOIC127P600X175-8N -> Package_TO_SOT_SMD:SOT-23
- moved J9 73.3 mm to (23.3, 52.0), turned to 270 degrees
- moved FB1 23.1 mm to (41.2, 40.6)
- moved G*** 18.6 mm to (54.3, 53.5)
- moved C1 15.7 mm to (36.3, 43.5)
- moved U1 15.6 mm to (43.7, 36.0), turned to 0 degrees
- moved R20 14.4 mm to (46.2, 35.5), turned to 90 degrees
- moved R3 13.9 mm to (42.3, 56.0), turned to 180 degrees
- moved F1 13.3 mm to (37.1, 39.7), turned to 0 degrees
- moved C3 13.2 mm to (41.2, 37.0), turned to 90 degrees
- moved R2 12.6 mm to (42.3, 54.5), turned to 180 degrees
- moved C4 12.6 mm to (42.3, 52.9), turned to 0 degrees
- moved C2 12.2 mm to (33.9, 43.5)
- moved Q1 11.7 mm to (32.3, 39.2)
- moved R21 11.7 mm to (43.8, 38.5), turned to 180 degrees
- moved R1 10.8 mm to (38.8, 43.5), turned to 90 degrees
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Connections:
- F1 pad 1: VCC -> VS
- FB1 pad 2: VS -> Net-(F1-Pad2)
- H1 pad 1: GND -> Net-(H1-Pad1)
- H2 pad 1: GND -> Net-(H2-Pad1)
- H3 pad 1: GND -> Net-(H3-Pad1)
- H4 pad 1: GND -> Net-(H4-Pad1)
- J9 pad 1: VBUS -> GND
- J9 pad 2: GND -> +3V3
- Q1 pad 1: VS -> GND
- Q1 pad 3: VS -> VCC
- U7 pad 32: Net-(U7-Pad32) -> MAGD_DRDY
- U7 pad 33: Net-(U7-Pad33) -> MAG_INT
- U7 pad 34: MAGD_DRDY -> TIM3_CH3
- U7 pad 35: MAG_INT -> TIM3_CH4
- U7 pad 43: Net-(U7-Pad43) -> TIM1_CH3
- U7 pad 44: Net-(U7-Pad44) -> TIM1_CH4
- U7 pad 57: Net-(U7-Pad57) -> GPIO_A
- U7 pad 58: Net-(U7-Pad58) -> GPIO_B
- U7 pad 83: Net-(U7-Pad83) -> ACC_INT
- U7 pad 84: Net-(U7-Pad84) -> GYR_INT
- U7 pad 90: ACC_INT -> TIM3_CH1
- U7 pad 91: GYR_INT -> TIM3_CH2
Routing:
- net TIM3_CH2: track 0.00 -> 79.4 mm, vias 0 -> 2
- net TIM3_CH1: track 0.00 -> 78.0 mm, vias 0 -> 2
- net TIM1_CH3: track 0.00 -> 71.5 mm, vias 0 -> 2
- net TIM1_CH4: track 0.00 -> 71.0 mm, vias 0 -> 2
- net TIM3_CH3: track 0.00 -> 60.4 mm, vias 0 -> 2
- net TIM3_CH4: track 0.00 -> 60.3 mm, vias 0 -> 2
- net GPIO_B: track 0.00 -> 42.2 mm, vias 0 -> 2
- net GND: track 156.5 -> 196.9 mm, vias 192 -> 92
- net GPIO_A: track 0.00 -> 37.8 mm, vias 0 -> 2
- net VS: track 122.4 -> 91.8 mm
- net +3V3: track 145.0 -> 115.5 mm, vias 48 -> 46
- net I2C1_SDA: track 50.5 -> 32.0 mm
- net I2C1_SCL: track 49.1 -> 31.3 mm
- net VDD: track 9.38 -> 17.6 mm, vias 0 -> 2
- net UART4_TX: track 21.1 -> 29.1 mm
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- removed copper zone on B.Cu, net GND
- removed copper zone on F.Cu, net GND
Other:
- board text added: "RC"
- board text added: "S"
- board text removed: "VI-MMXX"
